File: ESP32-S3.kicad_sch (KiCad schematic)
At the start: 19 parts, among them J1 USB_C_Receptacle_USB2.0_16P, U1 USBLC6-2SC6, U2 AMS1117-3.3, U3 ESP32-S3-WROOM-1

Commit message: can, usb
Parts:
- added C10, C9: 100n, Capacitor_SMD:C_0805_2012Metric, symbol Device:C
- added C11, C12: 100nF, Capacitor_SMD:C_0805_2012Metric, symbol Device:C
- added C13: 4.7nF, Capacitor_SMD:C_0805_2012Metric, symbol Device:C
- added C14: 1uF, Capacitor_SMD:C_0805_2012Metric, symbol Device:C
- added C15, C16: 10uF, Capacitor_SMD:C_0805_2012Metric, symbol Device:C
- added J2, J3: CAN_JST-GH, Connector_JST:JST_GH_SM04B-GHS-TB_1x04-1MP_P1.25mm, symbol Connector_Generic:Conn_01x04
- added JP1: SolderJumper_2_Open, Jumper:SolderJumper-2_P1.3mm_Open_RoundedPad1.0x1.5mm, symbol Jumper:SolderJumper_2_Open
- added R10, R9: 60, Resistor_SMD:R_0805_2012Metric, symbol Device:R
- added R5, R7: 10k, symbol Device:R
- added R6, R8: 100, symbol Device:R
- added SW1, SW2: SW_Push, symbol Switch:SW_Push
- added U4: TJA1051T/3, Package_SO:SOIC-8_3.9x4.9mm_P1.27mm, symbol Interface_CAN_LIN:TJA1051T
- added U5: AP3602A, Package_TO_SOT_SMD:SOT-23-6, symbol Diode_Inc:AP3602A
- R4: value 75 -> 100
Connections:
- net +3V3: now also C15.1, R5.1, R7.1, U5.3 (~{SHDN}), U5.5 (VIN)
- net +5V: now also J2.1 (Pin_1), J3.1 (Pin_1)
- net GND: now also C10.2, C11.2, C12.2, C13.2, C15.2, C16.2, C9.2, J2.4 (Pin_4), J3.4 (Pin_4), SW1.1, SW2.1, U4.2 (GND), U4.8 (S), U5.2 (GND)
- net USB_D+: now also U3.14 (USB_D+)
- net USB_D-: now also U3.13 (USB_D-)
- net D+: now reaches J1.A6 (D+), J1.A7 (D-), J1.B6 (D+), J1.B7 (D-), U1.1 (I/O1), U1.3 (I/O2)
- net BOOT: now reaches U3.27 (IO0)
- net BOOT: now also C10.1, R8.2
- net EN: now reaches U3.3 (EN)
- net EN: now also C9.1, R6.2
- net CAN_TX: now reaches U3.4 (IO4)
- net CAN_TX: now also U4.1 (TXD)
- net CAN_RX: now reaches U3.5 (IO5)
- net CAN_RX: now also U4.4 (RXD)
- new net: C14.1, U5.6 (C+)
- new net: C14.2, U5.4 (C-)
- new net: R5.2, R6.1, SW1.2
- new net: R7.2, R8.1, SW2.2
- new net: C13.1, R10.1, R9.2
- new net: JP1.2, R9.1
- new net +5V_CAN: C11.1, C12.1, C16.1, U4.3 (VCC), U4.5 (VIO), U5.1 (5VO)
- new net CANH: J2.2 (Pin_2), J3.2 (Pin_2), JP1.1, U4.7 (CANH)
- new net CANL: J2.3 (Pin_3), J3.3 (Pin_3), R10.2, U4.6 (CANL)
Other:
- note added: "CAN"
- note added: "ESP32-S3"
- note added: "Reset Buttons"
- moved on the sheet: C3, C4, C5, C6, C7, C8, D3, R4, U2, U3
