File: untitled.kicad_sch (KiCad schematic)
At the start: 0 parts

Commit message: Updated ready for review schematic
Changed lines of the file:
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@@
 	)
 	(rectangle
-		(start 113.03 146.05)
-		(end 127 157.48)
+		(start 71.12 133.35)
+		(end 85.09 144.78)
 		(stroke
 			(width 0)
