File: .claude/pre_footprint_audit_backup.kicad_sch (KiCad schematic)
At the start: 64 parts, among them J1 USB_C_Receptacle_USB2.0_16P, J10 5055670271, J12 5054482071, J2 5055670271, J3 SM04B-GHS-TB, J4 XT30 (right-angle), J5 SM04B-GHS-TB, J6 5055670271, J7 5055670271, J8 5055670271, Q1 DMP3098L-7, SW1 B3U-1000P, SW2 B3U-1000P, U1 USBLC6-2SC6, U2 AMS1117-3.3, U3 ESP32-S3-WROOM-1, U4 TJA1051T/3, U5 AP3602A, U6 LMR33630

Commit message: Updated ready for review schematic
Parts:
- C10, C11, C12, C13, C14, C7, C9: footprint Capacitor_SMD:C_0603_1608Metric -> Capacitor_SMD:C_0805_2012Metric
- C18, C4, C5: footprint Capacitor_SMD:C_0805_2012Metric -> Capacitor_SMD:C_0603_1608Metric
- L1: footprint Footprints:L_Wurth_WE-PD-1260 -> (none)
- R12, R13, R14: footprint Resistor_SMD:R_0603_1608Metric -> Resistor_SMD:R_0402_1005Metric
- SW1, SW2: value B3U-1000P -> SW_Push; footprint Button_Switch_SMD:SW_SPST_B3U-1000P -> (none)
- U6: footprint Footprints:DDA0008J -> Package_SO:HSOP-8_3.9x4.9mm_P1.27mm
Connections:
- net D- is gone; now on net D+: J1.A7 (D-), J1.B7 (D-), U1.1 (I/O1)
- net +3V3: no longer C12.1, U4.5 (VIO)
- net +5V_CAN: now also C12.1, U4.5 (VIO)
- net GPIO39: no longer J12.15
- net GPIO41: now reaches U3.34 (IO41)
- net GPIO42: now reaches U3.35 (IO42)
- no-connect marks 17 -> 2
Other:
- moved on the sheet: J12
